File: amiga_a520_svid.sch (KiCad schematic (older format))
At the start: 94 parts, among them J1 Conn_01x16, J10 Y, J11 Y, J12 COMP, J13 COMP, J14 GND, J15 GND, J16 Cr, J17 Cr, J18 LUMA, J19 LUMA, J2 Y, J20 GND, J21 GND, J22 GND, J23 GND, J24 Cb, J25 Cb, J26 CRMA, J27 CRMA, J28 GND, J29 GND, J3 Cr, J30 GND, J31 GND, J4 Cb, J5 COMP, J6 LUMA, J7 CRMA, J8 FU, J9 FU, Q1 2N3906, U1 AD8056ANZ, U2 AD8056ANZ, U3 AD8056ANZ, U4 AD724JRZ-R7

Commit message: Fixes after 1st prototype :)
- Swapped OPAMP outputs :(
- More careful AD724 implementation
- MORE SMD! Through hole without metallization is a pain!
Parts:
- removed Q1: 2N3906, Package_TO_SOT_THT:TO-92_Inline, symbol Transistor_BJT:2N3906
- added C41: 100n, Capacitor_SMD:C_1206_3216Metric_Pad1.33x1.80mm_HandSolder, symbol Device:C
- added C42, C43: 10u, Capacitor_SMD:CP_Elec_5x5.4, symbol Device:CP
- added C44: 32p, Capacitor_SMD:C_1206_3216Metric_Pad1.33x1.80mm_HandSolder, symbol Device:C
- added C48, C49, C50: 220u, Capacitor_SMD:CP_Elec_6.3x7.7, symbol Device:CP
- added L3: 3.3uH, Inductor_THT:L_Axial_L7.0mm_D3.3mm_P10.16mm_Horizontal_Fastron_MICC, symbol Device:L
- added R50, R51: 5k, Resistor_SMD:R_1206_3216Metric_Pad1.30x1.75mm_HandSolder, symbol Device:R
- added Y1: 17.734MHz, Crystal:Resonator-2Pin_W10.0mm_H5.0mm, symbol Device:Crystal
- C1, C13, C14, C2, C5, C6: footprint Capacitor_THT:C_Disc_D5.0mm_W2.5mm_P5.00mm -> Capacitor_SMD:C_1206_3216Metric_Pad1.33x1.80mm_HandSolder
- C10, C11, C12, C9: value 4.7u -> 10u; footprint Capacitor_THT:CP_Radial_D5.0mm_P2.50mm -> Capacitor_SMD:CP_Elec_5x5.4
- C40: renamed from C30; footprint Capacitor_THT:C_Disc_D5.0mm_W2.5mm_P5.00mm -> Capacitor_SMD:C_1206_3216Metric_Pad1.33x1.80mm_HandSolder
- C45: renamed from Co1; footprint Capacitor_THT:C_Disc_D5.0mm_W2.5mm_P5.00mm -> Capacitor_SMD:C_1206_3216Metric_Pad1.33x1.80mm_HandSolder
- C46: renamed from Co2; footprint Capacitor_THT:C_Disc_D5.0mm_W2.5mm_P5.00mm -> Capacitor_SMD:C_1206_3216Metric_Pad1.33x1.80mm_HandSolder
- C47: renamed from Co3; footprint Capacitor_THT:C_Disc_D5.0mm_W2.5mm_P5.00mm -> Capacitor_SMD:C_1206_3216Metric_Pad1.33x1.80mm_HandSolder
- J1: footprint Connector_PinSocket_1.27mm:PinSocket_1x16_P1.27mm_Vertical -> Connector_PinHeader_1.27mm:PinHeader_1x16_P1.27mm_Vertical_SMD_Pin1Left
- L1, L2: value 1k@100MHz -> 3.3uH
- R1, R10, R11, R12, R13, R14, R15, R16, R17, R18, R19, R2, R20, R21, R22, R23, R24, R25, R26, R27, R28, R29, R3, R4, R5, R6, R7, R8, R9: footprint Resistor_SMD:R_1206_3216Metric -> Resistor_SMD:R_1206_3216Metric_Pad1.30x1.75mm_HandSolder
- R31: renamed from Ro1; footprint Resistor_SMD:R_1206_3216Metric -> Resistor_SMD:R_1206_3216Metric_Pad1.30x1.75mm_HandSolder
- R32: renamed from Ro2; footprint Resistor_SMD:R_1206_3216Metric -> Resistor_SMD:R_1206_3216Metric_Pad1.30x1.75mm_HandSolder
- R33: renamed from Ro3; footprint Resistor_SMD:R_1206_3216Metric -> Resistor_SMD:R_1206_3216Metric_Pad1.30x1.75mm_HandSolder
- R40: renamed from R35; value 1k -> 200; footprint Resistor_SMD:R_1206_3216Metric -> Resistor_SMD:R_1206_3216Metric_Pad1.30x1.75mm_HandSolder
- R41: renamed from R36; value 1k -> 200; footprint Resistor_SMD:R_1206_3216Metric -> Resistor_SMD:R_1206_3216Metric_Pad1.30x1.75mm_HandSolder
- R42: renamed from R33; value 1k -> 200; footprint Resistor_SMD:R_1206_3216Metric -> Resistor_SMD:R_1206_3216Metric_Pad1.30x1.75mm_HandSolder
- R43: renamed from R34; value 1k -> 200; footprint Resistor_SMD:R_1206_3216Metric -> Resistor_SMD:R_1206_3216Metric_Pad1.30x1.75mm_HandSolder
- R45: renamed from R31; value 1k -> 200; footprint Resistor_SMD:R_1206_3216Metric -> Resistor_SMD:R_1206_3216Metric_Pad1.30x1.75mm_HandSolder
- R46: renamed from R32; value 1k -> 200; footprint Resistor_SMD:R_1206_3216Metric -> Resistor_SMD:R_1206_3216Metric_Pad1.30x1.75mm_HandSolder
- R47: renamed from R37; footprint Resistor_SMD:R_1206_3216Metric -> Resistor_SMD:R_1206_3216Metric_Pad1.30x1.75mm_HandSolder
- R48: renamed from R38; footprint Resistor_SMD:R_1206_3216Metric -> Resistor_SMD:R_1206_3216Metric_Pad1.30x1.75mm_HandSolder
- R49: renamed from R39; footprint Resistor_SMD:R_1206_3216Metric -> Resistor_SMD:R_1206_3216Metric_Pad1.30x1.75mm_HandSolder
- renumbered Qa1 to Q1
Connections:
- net +5V: now also C42.1; no longer U4.14 (DPOS), U4.5 (ENCD)
- net Bb: now also U3.1 (OUT1); no longer U3.7 (OUT)
- net GND: now also C41.2, C42.2, C43.2, C44.1, Y1.1; no longer U4.12 (SELECT)
- net Gb: now also U2.1 (OUT1); no longer U2.7 (OUT)
- net Rb: now also U1.1 (OUT1); no longer U1.7 (OUT)
- net at R2.2, R8.1: now also U1.7 (OUT); no longer U1.1 (OUT1)
- net at U4.10 (COMP): now also C48.1; no longer R47.2
- net at U4.11 (LUMA): now also C50.1; no longer R49.2
- net at U4.6 (RIN): now also C47.2; no longer C45.1
- net at U4.8 (BIN): now also C45.2; no longer C47.2
- net at U4.9 (CRMA): now also C49.1; no longer R48.2
- net at R12.2, R18.1: now also U2.7 (OUT); no longer U2.1 (OUT1)
- net at R20.2, R26.1: now also U3.7 (OUT); no longer U3.1 (OUT1)
- net R: now reaches J1.1 (Pin_1), R31.2
- net VDC: now reaches C11.1, J1.13 (Pin_13), L1.2
- net VDC: now also L3.2
- net at R45.1, R46.2: now also C47.1; no longer C45.2
- net at R40.1, R41.2: now also C45.1; no longer C47.1
- net -5V renamed -12V
- net BURST: no longer names the net of U4.3 (FIN)
- net BURST: now also C44.2, Y1.2; no longer J1.16 (Pin_16)
- new net: R50.1, U4.12 (SELECT)
- new net: C41.1, C43.1, L3.1, R50.2, R51.2, U4.14 (DPOS)
- new net: R51.1, U4.5 (ENCD)
- new net: C48.2, R47.2
- new net: C49.2, R48.2
- new net: C50.2, R49.2
- no-connect marks 0 -> 1
Other:
- moved on the sheet: C1, C13, C14, C2, C40, C45, C46, C47, C5, C6, J10, J11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
